Commit message: 修改：     .vscode/settings.json 	修改：     build/CMakeCache.txt 	修改：     build/CMakeFiles/Makefile.cmake 	修改：     build/CMakeFiles/Makefile2 	修改：     build/CMakeFiles/TargetDirectories.txt 	修改：     build/CMakeFiles/progress.marks 	修改：     build/CTestTestfile.cmake 	修改：     build/Makefile 	修改：     build/catkin_generated/order_packages.cmake 	修改：     build/catkin_make.cache 	修改：     build/cmake_install.cmake 	修改：     build/control_turtle/CMakeFiles/control_param.dir/progress.make 	修改：     build/control_turtle/CMakeFiles/control_pub.dir/progress.make 	修改：     build/control_turtle/CMakeFiles/control_sub.dir/progress.make 	修改：     build/control_turtle/CMakeFiles/progress.marks 	修改：     build/gtest/googlemock/CMakeFiles/gmock.dir/progress.make 	修改：     build/gtest/googlemock/CMakeFiles/gmock_main.dir/progress.make 	修改：     build/gtest/googlemock/gtest/CMakeFiles/gtest.dir/progress.make 	修改：     build/gtest/googlemock/gtest/CMakeFiles/gtest_main.dir/progress.make 	修改：     build/head_study/CMakeFiles/hello.dir/progress.make 	修改：     build/head_study/CMakeFiles/progress.marks 	修改：     build/head_study/Makefile 	修改：     build/plumbing_param_server/CMakeFiles/demo04_param_del.dir/progress.make 	修改：     build/plumbing_param_server/CMakeFiles/demo04_param_get.dir/progress.make 	修改：     build/plumbing_param_server/CMakeFiles/demo04_param_set.dir/progress.make 	修改：     build/plumbing_param_server/CMakeFiles/progress.marks 	修改：     build/plumbing_pubsub/CMakeFiles/demo01_pub.dir/progress.make 	修改：     build/plumbing_pubsub/CMakeFiles/demo01_sub.dir/progress.make 	修改：     build/plumbing_pubsub/CMakeFiles/demo02_pub_person.dir/progress.make 	修改：     build/plumbing_pubsub/CMakeFiles/demo02_sub_person.dir/progress.make 	修改：     build/plumbing_pubsub/CMakeFiles/plumbing_pubsub_generate_messages_cpp.dir/progress.make 	修改：     build/plumbing_pubsub/CMakeFiles/plumbing_pubsub_generate_messages_eus.dir/progress.make 	修改：     build/plumbing_pubsub/CMakeFiles/plumbing_pubsub_generate_messages_lisp.dir/progress.make 	修改：     build/plumbing_pubsub/CMakeFiles/plumbing_pubsub_generate_messages_nodejs.dir/progress.make 	修改：     build/plumbing_pubsub/CMakeFiles/plumbing_pubsub_generate_messages_py.dir/progress.make 	修改：     build/plumbing_pubsub/CMakeFiles/progress.marks 	修改：     build/plumbing_server_client/CMakeFiles/demo03_client.dir/progress.make 	修改：     build/plumbing_server_client/CMakeFiles/demo03_server.dir/progress.make 	修改：     build/plumbing_server_client/CMakeFiles/plumbing_server_client_generate_messages_cpp.dir/progress.make 	修改：     build/plumbing_server_client/CMakeFiles/plumbing_server_client_generate_messages_eus.dir/progress.make 	修改：     build/plumbing_server_client/CMakeFiles/plumbing_server_client_generate_messages_lisp.dir/progress.make 	修改：     build/plumbing_server_client/CMakeFiles/plumbing_server_client_generate_messages_nodejs.dir/progress.make 	修改：     build/plumbing_server_client/CMakeFiles/plumbing_server_client_generate_messages_py.dir/progress.make 	修改：     build/plumbing_server_client/CMakeFiles/progress.marks 	修改：     build/read_data/CMakeFiles/progress.marks 	修改：     build/read_data/CMakeFiles/read_data_scan_to_pointclod2_converter_node.dir/progress.make 	修改：     build/read_data/CMakeFiles/read_imu.dir/progress.make 	修改：     build/read_data/CMakeFiles/read_pcl.dir/progress.make 	修改：     build/ros_apis/CMakeFiles/apis_log.dir/progress.make 	修改：     build/ros_apis/CMakeFiles/apis_pub.dir/progress.make 	修改：     build/ros_apis/CMakeFiles/apis_sub.dir/progress.make 	修改：     build/ros_apis/CMakeFiles/apis_times.dir/progress.make 	修改：     build/ros_apis/CMakeFiles/progress.marks 	修改：     build/rosbag_rw/CMakeFiles/bag_read.dir/progress.make 	修改：     build/rosbag_rw/CMakeFiles/bag_write.dir/progress.make 	修改：     build/rosbag_rw/CMakeFiles/progress.marks 	修改：     build/src_study/CMakeFiles/head_src.dir/progress.make 	修改：     build/src_study/CMakeFiles/use_hello.dir/progress.make 	修改：     build/tf2_dynamic/CMakeFiles/dynamic_pub.dir/progress.make 	修改：     build/tf2_dynamic/CMakeFiles/dynamic_sub.dir/progress.make 	修改：     build/tf2_dynamic/CMakeFiles/progress.marks 	修改：     build/tf2_static/CMakeFiles/progress.marks 	修改：     build/tf2_static/CMakeFiles/static_pub.dir/progress.make 	修改：     build/tf2_static/CMakeFiles/static_sub.dir/progress.make 	修改：     build/tf2s/CMakeFiles/tf2s_sub.dir/progress.make 	修改：     build/tf_turtle/CMakeFiles/create_turtle.dir/progress.make 	修改：     build/tf_turtle/CMakeFiles/progress.marks 	修改：     build/tf_turtle/CMakeFiles/pub_tf.dir/progress.make 	修改：     build/tf_turtle/CMakeFiles/sub_turtle.dir/progress.make 	新文件：   build/urdf_demo/CMakeFiles/roscpp_generate_messages_cpp.dir/DependInfo.cmake 	新文件：   build/urdf_demo/CMakeFiles/roscpp_generate_messages_cpp.dir/build.make 	新文件：   build/urdf_demo/CMakeFiles/roscpp_generate_messages_cpp.dir/cmake_clean.cmake 	新文件：   build/urdf_demo/CMakeFiles/roscpp_generate_messages_cpp.dir/depend.internal 	新文件：   build/urdf_demo/CMakeFiles/roscpp_generate_messages_cpp.dir/depend.make 	新文件：   build/urdf_demo/CMakeFiles/roscpp_generate_messages_cpp.dir/progress.make 	新文件：   build/urdf_demo/CMakeFiles/roscpp_generate_messages_eus.dir/DependInfo.cmake 	新文件：   build/urdf_demo/CMakeFiles/roscpp_generate_messages_eus.dir/build.make 	新文件：   build/urdf_demo/CMakeFiles/roscpp_generate_messages_eus.dir/cmake_clean.cmake 	新文件：   build/urdf_demo/CMakeFiles/roscpp_generate_messages_eus.dir/depend.internal 	新文件：   build/urdf_demo/CMakeFiles/roscpp_generate_messages_eus.dir/depend.make 	新文件：   build/urdf_demo/CMakeFiles/roscpp_generate_messages_eus.dir/progress.make 	新文件：   build/urdf_demo/CMakeFiles/roscpp_generate_messages_lisp.dir/DependInfo.cmake 	新文件：   build/urdf_demo/CMakeFiles/roscpp_generate_messages_lisp.dir/build.make 	新文件：   build/urdf_demo/CMakeFiles/roscpp_generate_messages_lisp.dir/cmake_clean.cmake 	新文件：   build/urdf_demo/CMakeFiles/roscpp_generate_messages_lisp.dir/depend.internal 	新文件：   build/urdf_demo/CMakeFiles/roscpp_generate_messages_lisp.dir/depend.make 	新文件：   build/urdf_demo/CMakeFiles/roscpp_generate_messages_lisp.dir/progress.make 	新文件：   build/urdf_demo/CMakeFiles/roscpp_generate_messages_nodejs.dir/DependInfo.cmake 	新文件：   build/urdf_demo/CMakeFiles/roscpp_generate_messages_nodejs.dir/build.make 	新文件：   build/urdf_demo/CMakeFiles/roscpp_generate_messages_nodejs.dir/cmake_clean.cmake 	新文件：   build/urdf_demo/CMakeFiles/roscpp_generate_messages_nodejs.dir/depend.internal 	新文件：   build/urdf_demo/CMakeFiles/roscpp_generate_messages_nodejs.dir/depend.make 	新文件：   build/urdf_demo/CMakeFiles/roscpp_generate_messages_nodejs.dir/progress.make 	新文件：   build/urdf_demo/CMakeFiles/roscpp_generate_messages_py.dir/DependInfo.cmake 	新文件：   build/urdf_demo/CMakeFiles/roscpp_generate_messages_py.dir/build.make 	新文件：   build/urdf_demo/CMakeFiles/roscpp_generate_messages_py.dir/cmake_clean.cmake 	新文件：   build/urdf_demo/CMakeFiles/roscpp_generate_messages_py.dir/depend.internal 	新文件：   build/urdf_demo/CMakeFiles/roscpp_generate_messages_py.dir/depend.make 	新文件：   build/urdf_demo/CMakeFiles/roscpp_generate_messages_py.dir/progress.make 	新文件：   build/urdf_demo/CMakeFiles/rosgraph_msgs_generate_messages_cpp.dir/DependInfo.cmake 	新文件：   build/urdf_demo/CMakeFiles/rosgraph_msgs_generate_messages_cpp.dir/build.make 	新文件：   build/urdf_demo/CMakeFiles/rosgraph_msgs_generate_messages_cpp.dir/cmake_clean.cmake 	新文件：   build/urdf_demo/CMakeFiles/rosgraph_msgs_generate_messages_cpp.dir/depend.internal 	新文件：   build/urdf_demo/CMakeFiles/rosgraph_msgs_generate_messages_cpp.dir/depend.make 	新文件：   build/urdf_demo/CMakeFiles/rosgraph_msgs_generate_messages_cpp.dir/progress.make 	新文件：   build/urdf_demo/CMakeFiles/rosgraph_msgs_generate_messages_eus.dir/DependInfo.cmake 	新文件：   build/urdf_demo/CMakeFiles/rosgraph_msgs_generate_messages_eus.dir/build.make 	新文件：   build/urdf_demo/CMakeFiles/rosgraph_msgs_generate_messages_eus.dir/cmake_clean.cmake 	新文件：   build/urdf_demo/CMakeFiles/rosgraph_msgs_generate_messages_eus.dir/depend.internal 	新文件：   build/urdf_demo/CMakeFiles/rosgraph_msgs_generate_messages_eus.dir/depend.make 	新文件：   build/urdf_demo/CMakeFiles/rosgraph_msgs_generate_messages_eus.dir/progress.make 	新文件：   build/urdf_demo/CMakeFiles/rosgraph_msgs_generate_messages_lisp.dir/DependInfo.cmake 	新文件：   build/urdf_demo/CMakeFiles/rosgraph_msgs_generate_messages_lisp.dir/build.make 	新文件：   build/urdf_demo/CMakeFiles/rosgraph_msgs_generate_messages_lisp.dir/cmake_clean.cmake 	新文件：   build/urdf_demo/CMakeFiles/rosgraph_msgs_generate_messages_lisp.dir/depend.internal 	新文件：   build/urdf_demo/CMakeFiles/rosgraph_msgs_generate_messages_lisp.dir/depend.make 	新文件：   build/urdf_demo/CMakeFiles/rosgraph_msgs_generate_messages_lisp.dir/progress.make 	新文件：   build/urdf_demo/CMakeFiles/rosgraph_msgs_generate_messages_nodejs.dir/DependInfo.cmake 	新文件：   build/urdf_demo/CMakeFiles/rosgraph_msgs_generate_messages_nodejs.dir/build.make 	新文件：   build/urdf_demo/CMakeFiles/rosgraph_msgs_generate_messages_nodejs.dir/cmake_clean.cmake 	新文件：   build/urdf_demo/CMakeFiles/rosgraph_msgs_generate_messages_nodejs.dir/depend.internal 	新文件：   build/urdf_demo/CMakeFiles/rosgraph_msgs_generate_messages_nodejs.dir/depend.make 	新文件：   build/urdf_demo/CMakeFiles/rosgraph_msgs_generate_messages_nodejs.dir/progress.make 	新文件：   build/urdf_demo/CMakeFiles/rosgraph_msgs_generate_messages_py.dir/DependInfo.cmake 	新文件：   build/urdf_demo/CMakeFiles/rosgraph_msgs_generate_messages_py.dir/build.make 	新文件：   build/urdf_demo/CMakeFiles/rosgraph_msgs_generate_messages_py.dir/cmake_clean.cmake 	新文件：   build/urdf_demo/CMakeFiles/rosgraph_msgs_generate_messages_py.dir/depend.internal 	新文件：   build/urdf_demo/CMakeFiles/rosgraph_msgs_generate_messages_py.dir/depend.make 	新文件：   build/urdf_demo/CMakeFiles/rosgraph_msgs_generate_messages_py.dir/progress.make 	新文件：   build/urdf_demo/CMakeFiles/std_msgs_generate_messages_cpp.dir/DependInfo.cmake 	新文件：   build/urdf_demo/CMakeFiles/std_msgs_generate_messages_cpp.dir/build.make 	新文件：   build/urdf_demo/CMakeFiles/std_msgs_generate_messages_cpp.dir/cmake_clean.cmake 	新文件：   build/urdf_demo/CMakeFiles/std_msgs_generate_messages_cpp.dir/depend.internal 	新文件：   build/urdf_demo/CMakeFiles/std_msgs_generate_messages_cpp.dir/depend.make 	新文件：   build/urdf_demo/CMakeFiles/std_msgs_generate_messages_cpp.dir/progress.make 	新文件：   build/urdf_demo/CMakeFiles/std_msgs_generate_messages_eus.dir/DependInfo.cmake 	新文件：   build/urdf_demo/CMakeFiles/std_msgs_generate_messages_eus.dir/build.make 	新文件：   build/urdf_demo/CMakeFiles/std_msgs_generate_messages_eus.dir/cmake_clean.cmake 	新文件：   build/urdf_demo/CMakeFiles/std_msgs_generate_messages_eus.dir/depend.internal 	新文件：   build/urdf_demo/CMakeFiles/std_msgs_generate_messages_eus.dir/depend.make 	新文件：   build/urdf_demo/CMakeFiles/std_msgs_generate_messages_eus.dir/progress.make 	新文件：   build/urdf_demo/CMakeFiles/std_msgs_generate_messages_lisp.dir/DependInfo.cmake 	新文件：   build/urdf_demo/CMakeFiles/std_msgs_generate_messages_lisp.dir/build.make 	新文件：   build/urdf_demo/CMakeFiles/std_msgs_generate_messages_lisp.dir/cmake_clean.cmake 	新文件：   build/urdf_demo/CMakeFiles/std_msgs_generate_messages_lisp.dir/depend.internal 	新文件：   build/urdf_demo/CMakeFiles/std_msgs_generate_messages_lisp.dir/depend.make 	新文件：   build/urdf_demo/CMakeFiles/std_msgs_generate_messages_lisp.dir/progress.make 	新文件：   build/urdf_demo/CMakeFiles/std_msgs_generate_messages_nodejs.dir/DependInfo.cmake 	新文件：   build/urdf_demo/CMakeFiles/std_msgs_generate_messages_nodejs.dir/build.make 	新文件：   build/urdf_demo/CMakeFiles/std_msgs_generate_messages_nodejs.dir/cmake_clean.cmake 	新文件：   build/urdf_demo/CMakeFiles/std_msgs_generate_messages_nodejs.dir/depend.internal 	新文件：   build/urdf_demo/CMakeFiles/std_msgs_generate_messages_nodejs.dir/depend.make 	新文件：   build/urdf_demo/CMakeFiles/std_msgs_generate_messages_nodejs.dir/progress.make 	新文件：   build/urdf_demo/CMakeFiles/std_msgs_generate_messages_py.dir/DependInfo.cmake 	新文件：   build/urdf_demo/CMakeFiles/std_msgs_generate_messages_py.dir/build.make 	新文件：   build/urdf_demo/CMakeFiles/std_msgs_generate_messages_py.dir/cmake_clean.cmake 	新文件：   build/urdf_demo/CMakeFiles/std_msgs_generate_messages_py.dir/depend.internal 	新文件：   build/urdf_demo/CMakeFiles/std_msgs_generate_messages_py.dir/depend.make 	新文件：   build/urdf_demo/CMakeFiles/std_msgs_generate_messages_py.dir/progress.make 	新文件：   build/urdf_demo/CMakeFiles/urdf_demo_xacro_generated_to_devel_space_.dir/DependInfo.cmake 	新文件：   build/urdf_demo/CMakeFiles/urdf_demo_xacro_generated_to_devel_space_.dir/build.make 	新文件：   build/urdf_demo/CMakeFiles/urdf_demo_xacro_generated_to_devel_space_.dir/cmake_clean.cmake 	新文件：   build/urdf_demo/CMakeFiles/urdf_demo_xacro_generated_to_devel_space_.dir/depend.internal 	新文件：   build/urdf_demo/CMakeFiles/urdf_demo_xacro_generated_to_devel_space_.dir/depend.make 	新文件：   build/urdf_demo/CMakeFiles/urdf_demo_xacro_generated_to_devel_space_.dir/progress.make 	拷贝：     build/head_study/Makefile -> build/urdf_demo/Makefile 	新文件：   build/urdf_demo/catkin_generated/ordered_paths.cmake 	新文件：   src/gazebo_urdf/CMakeLists.txt 	新文件：   src/gazebo_urdf/package.xml 	修改：     src/urdf_demo/CMakeLists.txt 	新文件：   src/urdf_demo/config/hello.yaml 	新文件：   src/urdf_demo/launch/car.launch 	新文件：   src/urdf_demo/launch/demo.launch 	修改：     src/urdf_demo/launch/demo03.launch 	新文件：   src/urdf_demo/launch/demo04.launch 	新文件：   src/urdf_demo/launch/demo05.launch 	新文件：   src/urdf_demo/launch/demo06.launch 	修改：     src/urdf_demo/urdf/urdf/demo03_joint.urdf 	新文件：   src/urdf_demo/urdf/urdf/demo04_base_footprint.urdf 	新文件：   src/urdf_demo/urdf/urdf/demo05_test.urdf 	新文件：   src/urdf_demo/urdf/xacro/car.xacro 	新文件：   src/urdf_demo/urdf/xacro/demo.urdf 	新文件：   src/urdf_demo/urdf/xacro/demo.xacro 	新文件：   src/urdf_demo/urdf/xacro/demo_camera.xacro 	新文件：   src/urdf_demo/urdf/xacro/demo_laser.xacro

File: src/urdf_demo/urdf/urdf/demo03_joint.urdf (robot description, URDF)
Before this commit: robot mycar, 2 links, 1 joints
Links:
- link base_link: geometry visual box size=0.3 0.2 0.1
Joints:
- joint camera2baselink: origin xyz=0.2 0 0.075 rpy=0 0 0 -> xyz=0.1 0 0.05 rpy=0 0 0
